File: PCB/led.kicad_sch (KiCad schematic)
At the start: 36 parts

Commit message: v2: reversiblility for LHS and RHS
Parts:
- LED1, LED10, LED11, LED12, LED13, LED14, LED15, LED16, LED17, LED18, LED19, LED2, LED20, LED21, LED22, LED23, LED24, LED25, LED26, LED27, LED28, LED29, LED3, LED30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: footprint marbastlib-choc:LED_choc_6028R -> assets:LED_choc_6028R_Reversible_same_side
