File: PCB/matrix.kicad_sch (KiCad schematic)
At the start: 70 parts, among them K0 KC_ESC, K1 KC_GRV, K10 SW_Push, K11 KC_TAB, K12 KC_Q, K13 KC_W, K14 KC_E, K15 KC_R, K16 KC_T, K2 KC_1, K20 SW_Push, K21 KC_CAPS, K22 KC_A, K23 KC_S, K24 KC_D, K25 KC_F, K26 KC_G, K3 KC_2, K30 SW_Push, K31 KC_LSFT, K32 KC_Z, K33 KC_X, K34 KC_C, K35 KC_V, K36 KC_B, K4 KC_3, K40 SW_Push, K41 KC_LCTL, K42 KC_LGUI, K43 KC_LALT, K44 KC_FN, K45 KC_SPACE, K46 KC_SPACE, K5 KC_4, K6 KC_5

Commit message: v2: reversiblility for LHS and RHS
Parts:
- D0, D1, D10, D11, D12, D13, D14, D15, D16, D2, D20, D21, D22, D23, D24, D25, D26, D3, D30, D31, D32, D33, D34, D35, D36, D4, D40, D41, D42, D43, D44, D45, D46, D5, D6: footprint Diode_SMD:D_SOD-123 -> assets:D_SOD-123-Reversible
- K0, K1, K10, K11, K12, K13, K14, K15, K16, K2, K20, K21, K22, K23, K24, K25, K26, K3, K30, K31, K32, K33, K34, K35, K36, K4, K40, K41, K42, K43, K44, K45, K46, K5, K6: footprint Switch_Keyboard_Hotswap_Kailh:SW_Hotswap_Kailh_Choc_V1V2_1.00u -> assets:SW_choc_1u_reversible
