File: PCB/5x07.kicad_pcb (KiCad board)
At the start: 2 copper layers, 165.9 x 100.8 mm, 127 parts, among them J1 AVR-ISP-6, K0 KC_ESC, K1 KC_GRV, K10 SW_Push, K11 KC_TAB, K12 KC_Q, K13 KC_W, K14 KC_E, K15 KC_R, K16 KC_T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

Commit message: bugfix
Parts:
- added REF**: 5x07, assets:5x07, F.Cu at (69.8, 102.4)
- J1: footprint random-keyboard-parts:Reset_Pretty-Mask -> random-keyboard-parts:Reset_Pretty
Routing:
- net row4: track 203.2 -> 200.4 mm, vias 9 -> 8
- net col0: track 142.1 -> 140.7 mm
