File: PCB/5x07.kicad_sch (KiCad schematic)
At the start: 21 parts, among them J1 AVR-ISP-6, SW1 SW_Push, U1 ATmega32U4-A, U2 PRTR5V0U2X, Y1 16MHz

Commit message: bugfix
Parts:
- J1: footprint random-keyboard-parts:Reset_Pretty-Mask -> random-keyboard-parts:Reset_Pretty
Changed lines of the file:
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@@
       (effects (font (size 1.27 1.27)) (justify right))
     )
-    (property "Footprint" "random-keyboard-parts:Reset_Pretty-Mask" (id 2) (at 134.62 142.24 90)
+    (property "Footprint" "random-keyboard-parts:Reset_Pretty" (id 2) (at 134.62 142.24 90)
       (effects (font (size 1.27 1.27)) hide)
     )
@@
     )
     (path "/e5bff2ed-4470-4084-a621-480b9de3ee53"
-      (reference "J1") (unit 1) (value "AVR-ISP-6") (footprint "random-keyboard-parts:Reset_Pretty-Mask")
+      (reference "J1") (unit 1) (value "AVR-ISP-6") (footprint "random-keyboard-parts:Reset_Pretty")
     )
     (path "/4787577f-7d8a-45a2-be7c-203d64397828/b8baca79-5620-4f40-beee-40a42b9669e9"
